Commit message: Modify - initial pose of p73

File: robots/P73_description/urdf/p73.urdf (robot description, URDF)
Before this commit: robot P73, 33 links, 32 joints
Joints:
- joint L_Knee_Joint: limit lower=-3.14159 upper=3.14159 effort=300 velocity=100 -> lower=-3.14159 upper=0.0 effort=300 velocity=100
- joint R_Knee_Joint: limit lower=-3.14159 upper=3.14159 effort=300 velocity=100 -> lower=-3.14159 upper=0.0 effort=300 velocity=100

Commit message: lim's code backup

File: robots/P73_description/urdf/p73.urdf (robot description, URDF)
Before this commit: robot P73, 33 links, 32 joints
Joints:
- joint L_AnklePitch_Joint: limit lower=-3.14159 upper=3.14159 effort=300 velocity=100 -> lower=-3.14159 upper=3.14159 effort=300 velocity=10
- joint L_AnkleRoll_Joint: limit lower=-3.14159 upper=3.14159 effort=300 velocity=100 -> lower=-3.14159 upper=3.14159 effort=300 velocity=10
- joint L_Elbow_Joint: limit lower=-3.14159 upper=3.14159 effort=300 velocity=100 -> lower=-3.14159 upper=3.14159 effort=300 velocity=10
- joint L_HipPitch_Joint: limit lower=-3.14159 upper=3.14159 effort=300 velocity=100 -> lower=-3.14159 upper=3.14159 effort=300 velocity=10
- joint L_HipRoll_Joint: limit lower=-3.14159 upper=3.14159 effort=300 velocity=100 -> lower=-3.14159 upper=3.14159 effort=300 velocity=10
- joint L_HipYaw_Joint: limit lower=-3.14159 upper=3.14159 effort=300 velocity=100 -> lower=-3.14159 upper=3.14159 effort=300 velocity=10
- joint L_Knee_Joint: limit lower=-3.14159 upper=0.0 effort=300 velocity=100 -> lower=-3.14159 upper=0.0 effort=300 velocity=10
- joint L_ShoulderPitch_Joint: limit lower=-3.14159 upper=3.14159 effort=300 velocity=100 -> lower=-3.14159 upper=3.14159 effort=300 velocity=10
- joint L_ShoulderRoll_Joint: limit lower=-3.14159 upper=3.14159 effort=300 velocity=100 -> lower=-3.14159 upper=3.14159 effort=300 velocity=10
- joint L_ShoulderYaw_Joint: limit lower=-3.14159 upper=3.14159 effort=300 velocity=100 -> lower=-3.14159 upper=3.14159 effort=300 velocity=10
- joint L_WristPitch_Joint: limit lower=-3.14159 upper=3.14159 effort=300 velocity=100 -> lower=-3.14159 upper=3.14159 effort=300 velocity=10
- joint L_WristRoll_Joint: limit lower=-3.14159 upper=3.14159 effort=300 velocity=100 -> lower=-3.14159 upper=3.14159 effort=300 velocity=10
- joint L_WristYaw_Joint: limit lower=-3.14159 upper=3.14159 effort=300 velocity=100 -> lower=-3.14159 upper=3.14159 effort=300 velocity=10
- joint NeckPitch_Joint: limit lower=-3.14159 upper=3.14159 effort=300 velocity=100 -> lower=-3.14159 upper=3.14159 effort=300 velocity=10
- joint NeckRoll_Joint: limit lower=-3.14159 upper=3.14159 effort=300 velocity=100 -> lower=-3.14159 upper=3.14159 effort=300 velocity=10
- joint NeckYaw_Joint: limit lower=-3.14159 upper=3.14159 effort=300 velocity=100 -> lower=-3.14159 upper=3.14159 effort=300 velocity=10
- joint R_AnklePitch_Joint: limit lower=-3.14159 upper=3.14159 effort=300 velocity=100 -> lower=-3.14159 upper=3.14159 effort=300 velocity=10
- joint R_AnkleRoll_Joint: limit lower=-3.14159 upper=3.14159 effort=300 velocity=100 -> lower=-3.14159 upper=3.14159 effort=300 velocity=10
- joint R_Elbow_Joint: limit lower=-3.14159 upper=3.14159 effort=300 velocity=100 -> lower=-3.14159 upper=3.14159 effort=300 velocity=10
- joint R_HipPitch_Joint: limit lower=-3.14159 upper=3.14159 effort=300 velocity=100 -> lower=-3.14159 upper=3.14159 effort=300 velocity=10
- joint R_HipRoll_Joint: limit lower=-3.14159 upper=3.14159 effort=300 velocity=100 -> lower=-3.14159 upper=3.14159 effort=300 velocity=10
- joint R_HipYaw_Joint: limit lower=-3.14159 upper=3.14159 effort=300 velocity=100 -> lower=-3.14159 upper=3.14159 effort=300 velocity=10
- joint R_Knee_Joint: limit lower=-3.14159 upper=0.0 effort=300 velocity=100 -> lower=-3.14159 upper=0.0 effort=300 velocity=10
- joint R_ShoulderPitch_Joint: limit lower=-3.14159 upper=3.14159 effort=300 velocity=100 -> lower=-3.14159 upper=3.14159 effort=300 velocity=10
- joint R_ShoulderRoll_Joint: limit lower=-3.14159 upper=3.14159 effort=300 velocity=100 -> lower=-3.14159 upper=3.14159 effort=300 velocity=10
- joint R_ShoulderYaw_Joint: limit lower=-3.14159 upper=3.14159 effort=300 velocity=100 -> lower=-3.14159 upper=3.14159 effort=300 velocity=10
- joint R_WristPitch_Joint: limit lower=-3.14159 upper=3.14159 effort=300 velocity=100 -> lower=-3.14159 upper=3.14159 effort=300 velocity=10
- joint R_WristRoll_Joint: limit lower=-3.14159 upper=3.14159 effort=300 velocity=100 -> lower=-3.14159 upper=3.14159 effort=300 velocity=10
- joint R_WristYaw_Joint: limit lower=-3.14159 upper=3.14159 effort=300 velocity=100 -> lower=-3.14159 upper=3.14159 effort=300 velocity=10
- joint WaistPitch_Joint: limit lower=-3.14159 upper=3.14159 effort=300 velocity=100 -> lower=-3.14159 upper=3.14159 effort=300 velocity=10
- joint WaistRoll_Joint: limit lower=-3.14159 upper=3.14159 effort=300 velocity=100 -> lower=-3.14159 upper=3.14159 effort=300 velocity=10
- joint WaistYaw_Joint: limit lower=-3.14159 upper=3.14159 effort=300 velocity=100 -> lower=-3.14159 upper=3.14159 effort=300 velocity=10

Commit message: doolie help

File: robots/P73_description/urdf/p73.urdf (robot description, URDF)
Before this commit: robot P73, 33 links, 32 joints
Joints:
- joint L_Knee_Joint: limit lower=-3.14159 upper=0.0 effort=300 velocity=100 -> lower=-3.14159 upper=0.5 effort=300 velocity=100
- joint R_Knee_Joint: limit lower=-3.14159 upper=0.0 effort=300 velocity=100 -> lower=-3.14159 upper=0.5 effort=300 velocity=100
